File: circuits/PCB_Plate_v6.sch (EAGLE design)
At the start: 158 parts, among them J1 12.0V, J10 Router V+, J11 Router V-, J12 PCONN00012, J13 MPT-08-01-01-L-RA-LC, J14 IPL1-1XX-02-XXX-DH-K-XX-MKT, J15 BOARD00012, J16 TSW1X20, J17 TSW1X20, J2 9.0V, J26 BOARD00012, J27 BOARD00012, J28 BOARD00012, J29 BOARD00012, J3 VMOTOR_A2D, J30 BOARD00012, J31 BOARD00012, J32 BOARD00012, J33 BOARD00012, J34 BOARD00012, J35 BOARD00012, J36 BOARD00012, J37 BOARD00012, J38 BOARD00012, J39 BOARD00012, J4 5.0V, J40 BOARD00012, J41 BOARD00012, J42 BOARD00012, J43 BOARD00012, J44 BOARD00012, J45 BOARD00012, J46 PCONN00012, J47 BOARD00012, J5 3.3V, J53 IMOTOR_A2D, J58 BOARD00012, J59 BOARD00012, J6 BRAINSTEMSOCKET_FEMALE, J60 BOARD00012, J68 BOARD00012, J69 BOARD00012, J71 BOARD00012, J72 GPS15X, J73 BOARD00012, J74 BOARD00012, J75 BOARD00012, J76 BOARD00012, J77 BOARD00012, J78 BOARD00012, J79 INT2, J80 INT, J81 BOARD00012, J82 BOARD00012, J83 BOARD00012, J84 BOARD00012, J85 BOARD00012, J86 BOARD00012, J87 BOARD00012, J88 BOARD00012, J89 BOARD00012, J9 GND, J90 BOARD00012, J91 BOARD00012, J92 BOARD00012, J93 BOARD00012, J94 BOARD00012, J95 BOARD00012, J96 BOARD00008, J97 BOARD00008, M1 MOUNT-HOLE3.2, M2 MOUNT-HOLE3.2, M3 MOUNT-HOLE3.2, M4 MOUNT-HOLE3.2, Q1 IXTA52P10P, Q2 IXTA52P10P, Q3 IXTA52P10P, Q4 SI4322DY, Q5 SI4322DY, Q6 IXTA52P10P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

Commit message: checking in a fully routed top plate. can one take any longer?
Connections:
- new net N$80: J17.P$16, J6-B.P$16
- net BATTERY_MOTOR+_OUT: now also R4.2
- net BATTERY_MOTOR+_OUT_PRE: no longer R4.2
- net POWER_LIPO+_IN: no longer J17.P$16, J6-B.P$16
Other:
- moved on the sheet: D1, D2, R4
Changed lines of the file:
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@@
 <instance part="GND8" gate="G$1" x="81.28" y="111.76"/>
 <instance part="S1" gate="G$1" x="55.88" y="63.5" rot="R180"/>
-<instance part="D1" gate="G$1" x="114.3" y="116.84" rot="R90"/>
-<instance part="D2" gate="G$1" x="106.68" y="119.38" smashed="yes">
-<attribute name="NAME" x="102.616" y="116.586" size="1.27" layer="95" rot="R90"/>
+<instance part="D1" gate="G$1" x="193.04" y="116.84" rot="R90"/>
+<instance part="D2" gate="G$1" x="185.42" y="119.38" smashed="yes">
+<attribute name="NAME" x="181.356" y="116.586" size="1.27" layer="95" rot="R90"/>
 </instance>
-<instance part="R4" gate="G$1" x="106.68" y="132.08" rot="R90"/>
-<instance part="GND9" gate="G$1" x="106.68" y="99.06"/>
+<instance part="R4" gate="G$1" x="185.42" y="132.08" rot="R90"/>
+<instance part="GND9" gate="G$1" x="185.42" y="99.06"/>
 <instance part="Q2" gate="G$1" x="86.36" y="160.02" rot="R90"/>
 <instance part="R5" gate="G$1" x="124.46" y="76.2" rot="R90"/>
@@
 <net name="GND3" class="0">
 <segment>
-<wire x1="106.68" y1="114.3" x2="106.68" y2="109.22" width="0.1524" layer="91"/>
-<wire x1="106.68" y1="109.22" x2="106.68" y2="101.6" width="0.1524" layer="91"/>
-<wire x1="114.3" y1="114.3" x2="114.3" y2="109.22" width="0.1524" layer="91"/>
-<wire x1="114.3" y1="109.22" x2="106.68" y2="109.22" width="0.1524" layer="91"/>
-<junction x="106.68" y="109.22"/>
+<wire x1="185.42" y1="114.3" x2="185.42" y2="109.22" width="0.1524" layer="91"/>
+<wire x1="185.42" y1="109.22" x2="185.42" y2="101.6" width="0.1524" layer="91"/>
+<wire x1="193.04" y1="114.3" x2="193.04" y2="109.22" width="0.1524" layer="91"/>
+<wire x1="193.04" y1="109.22" x2="185.42" y2="109.22" width="0.1524" layer="91"/>
+<junction x="185.42" y="109.22"/>
 <pinref part="D2" gate="G$1" pin="C"/>
 <pinref part="GND9" gate="G$1" pin="GND3"/>
@@
 <net name="N$4" class="0">
 <segment>
-<wire x1="106.68" y1="127" x2="106.68" y2="124.46" width="0.1524" layer="91"/>
-<wire x1="106.68" y1="124.46" x2="106.68" y2="121.92" width="0.1524" layer="91"/>
-<wire x1="106.68" y1="124.46" x2="114.3" y2="124.46" width="0.1524" layer="91"/>
-<wire x1="114.3" y1="124.46" x2="114.3" y2="119.38" width="0.1524" layer="91"/>
-<junction x="106.68" y="124.46"/>
+<wire x1="185.42" y1="127" x2="185.42" y2="124.46" width="0.1524" layer="91"/>
+<wire x1="185.42" y1="124.46" x2="185.42" y2="121.92" width="0.1524" layer="91"/>
+<wire x1="185.42" y1="124.46" x2="193.04" y2="124.46" width="0.1524" layer="91"/>
+<wire x1="193.04" y1="124.46" x2="193.04" y2="119.38" width="0.1524" layer="91"/>
+<junction x="185.42" y="124.46"/>
 <pinref part="R4" gate="G$1" pin="1"/>
 <pinref part="D2" gate="G$1" pin="A"/>
@@
 <wire x1="152.4" y1="132.08" x2="152.4" y2="139.7" width="0.1524" layer="91"/>
 <wire x1="83.82" y1="139.7" x2="106.68" y2="139.7" width="0.1524" layer="91"/>
-<wire x1="106.68" y1="137.16" x2="106.68" y2="139.7" width="0.1524" layer="91"/>
 <wire x1="91.44" y1="162.56" x2="106.68" y2="162.56" width="0.1524" layer="91"/>
 <wire x1="106.68" y1="162.56" x2="106.68" y2="139.7" width="0.1524" layer="91"/>
@@
 <pinref part="U4" gate="-A" pin="VIN-"/>
 <pinref part="Q1" gate="G$1" pin="S"/>
-<pinref part="R4" gate="G$1" pin="2"/>
 <pinref part="Q2" gate="G$1" pin="S"/>
 <pinref part="R5" gate="G$1" pin="2"/>
@@
 <wire x1="167.64" y1="132.08" x2="167.64" y2="139.7" width="0.1524" layer="91"/>
 <wire x1="167.64" y1="139.7" x2="165.1" y2="139.7" width="0.1524" layer="91"/>
-<wire x1="167.64" y1="139.7" x2="175.26" y2="139.7" width="0.1524" layer="91"/>
+<wire x1="167.64" y1="139.7" x2="185.42" y2="139.7" width="0.1524" layer="91"/>
 <junction x="167.64" y="139.7"/>
-<label x="175.26" y="139.7" size="1.27" layer="95" xref="yes"/>
+<label x="200.66" y="139.7" size="1.27" layer="95" xref="yes"/>
 <pinref part="U4" gate="-A" pin="VIN+"/>
 <pinref part="R11" gate="G$1" pin="2"/>
 <pinref part="J97" gate="G$1" pin="P$1"/>
+<pinref part="R4" gate="G$1" pin="2"/>
+<wire x1="185.42" y1="139.7" x2="200.66" y2="139.7" width="0.1524" layer="91"/>
+<wire x1="185.42" y1="137.16" x2="185.42" y2="139.7" width="0.1524" layer="91"/>
+<junction x="185.42" y="139.7"/>
 </segment>
 </net>
@@
 <net name="POWER_LIPO+_IN" class="0">
 <segment>
-<wire x1="142.24" y1="121.92" x2="134.62" y2="121.92" width="0.1524" layer="91"/>
-<wire x1="134.62" y1="121.92" x2="114.3" y2="121.92" width="0.1524" layer="91"/>
-<junction x="134.62" y="121.92"/>
-<label x="142.24" y="121.92" size="1.27" layer="95" xref="yes"/>
-<pinref part="J6" gate="-B" pin="P$16"/>
-<pinref part="J17" gate="G$1" pin="P$16"/>
-</segment>
-<segment>
 <wire x1="71.12" y1="45.72" x2="68.58" y2="45.72" width="0.1524" layer="91"/>
 <wire x1="68.58" y1="45.72" x2="66.04" y2="45.72" width="0.1524" layer="91"/>
@@
 </segment>
 </net>
+<net name="N$80" class="0">
+<segment>
+<pinref part="J6" gate="-B" pin="P$16"/>
+<pinref part="J17" gate="G$1" pin="P$16"/>
+<wire x1="134.62" y1="121.92" x2="114.3" y2="121.92" width="0.1524" layer="91"/>
+</segment>
+</net>

Commit message: checking in board. revision a ready to go
Parts:
- removed C27: PCAPI00015, aAcroname:PCAPI00015
- removed C28: T491A106K010AT, aAcroname:T491A106K010AT
- removed C29, C30: PCAPI00016, aAcroname:PCAPI00016
- added C12: PCAPI00020, aAcroname:PCAPI00020
- added C13: T491D227K016ZT, aAcroname:T491D227K016ZT
- added C14: CAP_POLARIZED, aAcroname:CAP_POLARIZED
- added C15: PCAPI00023, aAcroname:PCAPI00023
- added C17: PCAPI00007, aAcroname:PCAPI00007
- added D10, D11, D4, D5, D6, D7, D8, D9: PDIOD00003, aAcroname:PDIOD00003
- added J100, J63, J99: GND, aAcroname:BOARD00003WVALUE
- added J48, J49, J50, J52, J55, J56, J57, J64, J65, J66, J67, J70: BOARD00012, aAcroname:BOARD00012
- added J51: (no value), aAcroname:BOARD00003WVALUE
- added J61: TSW1X20, aAcroname:TSW1X20
- added J62: VMOTOR_A2D, aAcroname:BOARD00003WVALUE
- added J98: 3.3V, aAcroname:BOARD00003WVALUE
- added M5, M6: MOUNT-HOLE3.2, aAcroname:MOUNT-HOLE3.2
- added M7: BRAINSTEM_MOUNT, avc:BRAINSTEM_MOUNT
- added R23, R24, R25, R26, R27, R28, R29, R30: PRESI00012, aAcroname:PRESI00012
- added U13: NC7SZ08M5X, aAcroname:NC7SZ08M5X
- C1: value T491D227K016ZT -> ECJ-1VC1H270J; device aAcroname:T491D227K016ZT -> aAcroname:ECJ-1VC1H270J; ACRONAME PCAPI00037 -> (none)
- C10, C4: value PCAPI00015 -> T491D227K016ZT; device aAcroname:PCAPI00015 -> aAcroname:T491D227K016ZT; ACRONAME (none) -> PCAPI00037
- C11: value PCAPI00015 -> T491D227K016ZT; device aAcroname:PCAPI00015 -> aAcroname:T491D227K016ZT; ACRONAME PCAPI00015 -> PCAPI00037; PARTNUM ECJ-1VB1E104K -> (none)
- C16: value PCAPI00020 -> PCAPI00015; device aAcroname:PCAPI00020 -> aAcroname:PCAPI00015
- C18: value T491B105K035AT -> PCAPI00015; device aAcroname:T491B105K035AT -> aAcroname:PCAPI00015
- C19: value PCAPI00005 -> PCAPI00016; device aAcroname:PCAPI00005 -> aAcroname:PCAPI00016
- C2: value T491D227K016ZT -> T491B105K035AT; device aAcroname:T491D227K016ZT -> aAcroname:T491B105K035AT; ACRONAME PCAPI00037 -> (none)
- C20: value PCAPI00020 -> PCAPI00016; device aAcroname:PCAPI00020 -> aAcroname:PCAPI00016
- C22: value T491B105K035AT -> T491A106K010AT; device aAcroname:T491B105K035AT -> aAcroname:T491A106K010AT
- C23: value ECJ-1VC1H270J -> PCAPI00015; device aAcroname:ECJ-1VC1H270J -> aAcroname:PCAPI00015
- C24: value PCAPI00007 -> T491A106K010AT; device aAcroname:PCAPI00007 -> aAcroname:T491A106K010AT
- C25: value PCAPI00023 -> PCAPI00015; device aAcroname:PCAPI00023 -> aAcroname:PCAPI00015
- C26: value T491A106K010AT -> PCAPI00015; device aAcroname:T491A106K010AT -> aAcroname:PCAPI00015; ACRONAME (none) -> PCAPI00015; PARTNUM (none) -> ECJ-1VB1E104K
- C3: value CAP_POLARIZED -> T491B105K035AT; device aAcroname:CAP_POLARIZED -> aAcroname:T491B105K035AT; CAPACITANCE ? -> (none)
- C5: value CAP_POLARIZED -> PCAPI00005; device aAcroname:CAP_POLARIZED -> aAcroname:PCAPI00005; CAPACITANCE ? -> (none)
- C8: value T491D227K016ZT -> PCAPI00020; device aAcroname:T491D227K016ZT -> aAcroname:PCAPI00020; ACRONAME PCAPI00037 -> (none)
- C9: value T491D227K016ZT -> CAP_POLARIZED; device aAcroname:T491D227K016ZT -> aAcroname:CAP_POLARIZED; ACRONAME PCAPI00037 -> (none); CAPACITANCE (none) -> ?
- D1: value BZT52C3V3-7-F -> PDIOD00001; device aAcroname:BZT52C3V3-7-F -> aAcroname:PDIOD00001
- D2: value PDIOD00001 -> BZT52C3V3-7-F; device aAcroname:PDIOD00001 -> aAcroname:BZT52C3V3-7-F
- J1: value 12.0V -> (none); device aAcroname:BOARD00003WVALUE -> aAcroname:BOARD00003
- J10: value Router V+ -> (none); device aAcroname:BOARD00003WVALUE -> aAcroname:BOARD00003
- J11: value Router V- -> (none); device aAcroname:BOARD00003WVALUE -> aAcroname:BOARD00003
- J12: value PCONN00012 -> GND; device aAcroname:PCONN00012 -> aAcroname:BOARD00003WVALUE; ACRONAME (none) -> -; NOTES (none) -> No Stuff; PARTNUM (none) -> -; UNITCOST (none) -> 0.0
- J13: value MPT-08-01-01-L-RA-LC -> (none); device avc:MPT-08-01-01-L-RA-LC -> aAcroname:BOARD00003
- J14: value IPL1-1XX-02-XXX-DH-K-XX-MKT -> 3.3V; device avc:IPL1-1XX-02-XXX-DH-K-XX-MKT -> aAcroname:BOARD00003WVALUE; ACRONAME (none) -> -; NOTES (none) -> No Stuff; PARTNUM (none) -> -; UNITCOST (none) -> 0.0
- J16: value TSW1X20 -> 5.0V; device aAcroname:TSW1X20 -> aAcroname:BOARD00003WVALUE
- J17: value TSW1X20 -> 3.3V; device aAcroname:TSW1X20 -> aAcroname:BOARD00003WVALUE; ACRONAME (none) -> -; NOTES (none) -> No Stuff; PARTNUM (none) -> -; UNITCOST (none) -> 0.0
- J18: value (none) -> 3.3V; device aAcroname:BOARD00003 -> aAcroname:BOARD00003WVALUE
- J19: value (none) -> 3.3V; device aAcroname:BOARD00003 -> aAcroname:BOARD00003WVALUE; ACRONAME (none) -> -; NOTES (none) -> No Stuff; PARTNUM (none) -> -; UNITCOST (none) -> 0.0
- J2: value 9.0V -> GND; ACRONAME (none) -> -; NOTES (none) -> No Stuff; PARTNUM (none) -> -; UNITCOST (none) -> 0.0
- J20, J23, J25: value (none) -> BOARD00012; device aAcroname:BOARD00003 -> aAcroname:BOARD00012
- J21: value (none) -> 9.0V; device aAcroname:BOARD00003 -> aAcroname:BOARD00003WVALUE
- J22: value (none) -> Router V+; device aAcroname:BOARD00003 -> aAcroname:BOARD00003WVALUE
- J24: value (none) -> Router V-; device aAcroname:BOARD00003 -> aAcroname:BOARD00003WVALUE
- J3: value VMOTOR_A2D -> GND; ACRONAME (none) -> -; NOTES (none) -> No Stuff; PARTNUM (none) -> -; UNITCOST (none) -> 0.0
- J30: value BOARD00012 -> GPS15X; device aAcroname:BOARD00012 -> avc:GPS15X
- J34: value BOARD00012 -> BRAINSTEMSOCKET_FEMALE; device aAcroname:BOARD00012 -> aAcroname:BRAINSTEMSOCKET_FEMALE
- J35: value BOARD00012 -> 12.0V; device aAcroname:BOARD00012 -> aAcroname:BOARD00003WVALUE
- J36: value BOARD00012 -> IPL1-1XX-02-XXX-DH-K-XX-MKT; device aAcroname:BOARD00012 -> avc:IPL1-1XX-02-XXX-DH-K-XX-MKT
- J37: value BOARD00012 -> TSW1X20; device aAcroname:BOARD00012 -> aAcroname:TSW1X20
- J39: value BOARD00012 -> INT; device aAcroname:BOARD00012 -> aAcroname:BOARD00003WVALUE
- J4: value 5.0V -> (none); device aAcroname:BOARD00003WVALUE -> aAcroname:BOARD00003
- J42, J43: value BOARD00012 -> BOARD00008; device aAcroname:BOARD00012 -> aAcroname:BOARD00008
- J44: value BOARD00012 -> MPT-08-01-01-L-RA-LC; device aAcroname:BOARD00012 -> avc:MPT-08-01-01-L-RA-LC
- J45: value BOARD00012 -> INT2; device aAcroname:BOARD00012 -> aAcroname:BOARD00003WVALUE
- J46: value PCONN00012 -> BOARD00012; device aAcroname:PCONN00012 -> aAcroname:BOARD00012
- J5: value 3.3V -> (none); device aAcroname:BOARD00003WVALUE -> aAcroname:BOARD00003
- J53: value IMOTOR_A2D -> BOARD00012; device aAcroname:BOARD00003WVALUE -> aAcroname:BOARD00012
- J54: device aAcroname:BOARD00003 -> aAcroname:BOARD00003WVALUE
- J59: value BOARD00012 -> IMOTOR_A2D; device aAcroname:BOARD00012 -> aAcroname:BOARD00003WVALUE
- J6: value BRAINSTEMSOCKET_FEMALE -> (none); device aAcroname:BRAINSTEMSOCKET_FEMALE -> aAcroname:BOARD00003
- J69: value BOARD00012 -> A1; device aAcroname:BOARD00012 -> aAcroname:BOARD00003WVALUE
- J7, J8: device aAcroname:BOARD00003WVALUE -> aAcroname:BOARD00003
- J72: value GPS15X -> A0; device avc:GPS15X -> aAcroname:BOARD00003WVALUE
- J75: value BOARD00012 -> D2; device aAcroname:BOARD00012 -> aAcroname:BOARD00003WVALUE
- J78: value BOARD00012 -> D1; device aAcroname:BOARD00012 -> aAcroname:BOARD00003WVALUE
- J79: value INT2 -> PCONN00012; device aAcroname:BOARD00003WVALUE -> aAcroname:PCONN00012
- J80: value INT -> BOARD00012; device aAcroname:BOARD00003WVALUE -> aAcroname:BOARD00012
- J82: value BOARD00012 -> D0; device aAcroname:BOARD00012 -> aAcroname:BOARD00003WVALUE
- J85: value BOARD00012 -> SCL; device aAcroname:BOARD00012 -> aAcroname:BOARD00003WVALUE
- J88: value BOARD00012 -> SDA; device aAcroname:BOARD00012 -> aAcroname:BOARD00003WVALUE
- J9: ACRONAME (none) -> -; NOTES (none) -> No Stuff; PARTNUM (none) -> -; UNITCOST (none) -> 0.0
- J91: value BOARD00012 -> GND; device aAcroname:BOARD00012 -> aAcroname:BOARD00003WVALUE
- J92: value BOARD00012 -> PCONN00012; device aAcroname:BOARD00012 -> aAcroname:PCONN00012
- J95: value BOARD00012 -> 5.0V; device aAcroname:BOARD00012 -> aAcroname:BOARD00003WVALUE
- J96, J97: value BOARD00008 -> BOARD00012; device aAcroname:BOARD00008 -> aAcroname:BOARD00012
- M2: ACRONAME (none) -> -; PARTNUM (none) -> -; SIZE (none) -> 3.2 mm
- Q1: value IXTA52P10P -> SI4322DY; device aAcroname:IXTA52P10P -> aAcroname:SI4322DY
- Q2: value IXTA52P10P -> SI4322DY; device aAcroname:IXTA52P10P -> aAcroname:SI4322DY; NOTES No Stuff -> (none)
- Q4: value SI4322DY -> IXTA52P10P; device aAcroname:SI4322DY -> aAcroname:IXTA52P10P; NOTES (none) -> No Stuff
- Q5: value SI4322DY -> IXTA52P10P; device aAcroname:SI4322DY -> aAcroname:IXTA52P10P
- R1: value ERJ-3EKF1780V -> PRESI00006; device aAcroname:ERJ-3EKF1780V -> aAcroname:PRESI00006
- R10: value PRESI00018 -> ERJ-3EKF1780V; device aAcroname:PRESI00018 -> aAcroname:ERJ-3EKF1780V
- R11: value PRESI00041 -> on; device aAcroname:PRESI00041 -> aAcroname:ERJ-3EKF3830V
- R12: value PRESI00006 -> PRESI00005; device aAcroname:PRESI00006 -> aAcroname:PRESI00005; ACRONAME PRESI00006 -> (none); PARTNUM ERJ-3EKF1001V -> (none); UNITCOST 0.006 -> (none)
- R13: value PRESI00006 -> PRESI00041; device aAcroname:PRESI00006 -> aAcroname:PRESI00041; ACRONAME PRESI00006 -> (none); PARTNUM ERJ-3EKF1001V -> (none); UNITCOST 0.006 -> (none)
- R15: value ERJ-2RKF1021X -> PRESI00018; device aAcroname:ERJ-2RKF1021X -> aAcroname:PRESI00018
- R16: value PRESI00006 -> ERJ-2RKF9101X; device aAcroname:PRESI00006 -> aAcroname:ERJ-2RKF9101X
- R17: value ERJ-3EKF1004V -> ERJ-2RKF1021X; device aAcroname:ERJ-3EKF1004V -> aAcroname:ERJ-2RKF1021X
- R18: value PRESI00006 -> PRESI00005; device aAcroname:PRESI00006 -> aAcroname:PRESI00005
- R2: value on -> PRESI00006; device aAcroname:ERJ-3EKF3830V -> aAcroname:PRESI00006
- R20, R21: ACRONAME (none) -> PRESI00006; PARTNUM (none) -> ERJ-3EKF1001V; UNITCOST (none) -> 0.006
- R22, R4: value PRESI00005 -> PRESI00006; device aAcroname:PRESI00005 -> aAcroname:PRESI00006
- R3: value PRESI00006 -> ERJ-3EKF1004V; device aAcroname:PRESI00006 -> aAcroname:ERJ-3EKF1004V
- R5: value ERJ-2RKF9101X -> PRESI00006; device aAcroname:ERJ-2RKF9101X -> aAcroname:PRESI00006
- R6: value ERJ-3EKF1780V -> on; device aAcroname:ERJ-3EKF1780V -> aAcroname:ERJ-3EKF3830V
- R7: value on -> ERJ-3EKF1780V; device aAcroname:ERJ-3EKF3830V -> aAcroname:ERJ-3EKF1780V
- S2: value PMISC00005 -> EVQ-PE104K; device aAcroname:PMISC00005 -> aAcroname:EVQ-PE104K
- S3: value EVQ-PE104K -> PMISC00005; device aAcroname:EVQ-PE104K -> aAcroname:PMISC00005
- U1: value (none) -> LM3150; device aAcroname:LM1084IS-ADJ -> avc:LM3150
- U10: value ADS7828E -> I2C_DIO_EXPANDER; device aAcroname:ADS7828E -> aAcroname:I2C_DIO_EXPANDER
- U11: value CMPS10 -> MCP1416; device avc:CMPS10 -> aAcroname:MCP1416; PARTNUM (none) -> MCP1415T-E/OT
- U12: value ADXL335 -> LTV-356T; device avc:ADXL335 -> aAcroname:LTV-356T
- U4: value PCHIP00026 -> (none); device aAcroname:PCHIP00026 -> aAcroname:LM1084IS-ADJ
- U5: value MCP1416 -> L3G4200DTR; device aAcroname:MCP1416 -> avc:L3G4200DTR; PARTNUM MCP1415T-E/OT -> (none)
- U6: value LM3150 -> ADXL335; device avc:LM3150 -> avc:ADXL335
- U7: value LTV-356T -> CMPS10; device aAcroname:LTV-356T -> avc:CMPS10
- U8: value NC7SZ08M5X -> PCHIP00026; device aAcroname:NC7SZ08M5X -> aAcroname:PCHIP00026
- U9: value L3G4200DTR -> ADS7828E; device avc:L3G4200DTR -> aAcroname:ADS7828E
Connections:
- removed net N$11: J36.P$1
- removed net N$6 (its old number): R6.1, R7.2, U2.ADJ/GND
- new net GP2_D1: J67.P$1, J78.P$3
- new net GP2_D2: J66.P$1, J75.P$3
- new net I2C_CH0: J71.P$2, J79.P$9
- new net I2C_CH1: J74.P$2, J79.P$10
- new net I2C_CH2: J77.P$2, J79.P$11
- new net I2C_CH3: J79.P$12, J81.P$2
- new net I2C_CH4: J84.P$2, J92.P$9
- new net I2C_CH5: J87.P$2, J92.P$10
- new net I2C_CH6: J90.P$2, J92.P$11
- new net I2C_CH7: J92.P$12, J94.P$2
- new net N$101: R26.1, U10G$1.P3
- new net N$102: R30.1, U10G$1.P4
- new net N$104: R29.1, U10G$1.P5
- new net N$105: R28.1, U10G$1.P6
- new net N$108: R27.1, U10G$1.P7
- new net N$7: R6.2, R7.1, U2.ADJ/GND
- new net N$81: R23.1, U10G$1.P0
- new net N$82: D5.C, R24.2
- new net N$83: D6.C, R25.2
- new net N$84: D7.C, R26.2
- new net N$88: D11.C, R30.2
- new net N$89: D10.C, R29.2
- new net N$92: D9.C, R28.2
- new net N$93: D8.C, R27.2
- new net N$94: R24.1, U10G$1.P1
- new net N$95: R25.1, U10G$1.P2
- net !RESET: now also J34-A.P$1, J37.P$1, S2.S; no longer J16.P$1, J6-A.P$1, S3.S
- net 12.0V: now also C13.+, J31.P$1, J32.P$1, J33.P$1, J35.P$3, J44.5@0, J44.5@1, J44.5@2, J44.5@3, J44.5@4, J44.5@5, U4.INPUT; no longer C1.+, J1.P$3, J13.5@0, J13.5@1, J13.5@2, J13.5@3, J13.5@4, J13.5@5, J15.P$1, J81.P$1, J82.P$1, U1.INPUT
- net 3V3: now also C23.2, C24.+, C25.1, C26.2, D10.A, D11.A, D4.A, D5.A, D6.A, D7.A, D8.A, D9.A, J14.P$3, J15.P$1, J17.P$3, J18.P$3, J19.P$3, J29.P$2, J34-B.P$18, J34-B.P$19, J38.P$2, J46.P$1, J50.P$2, J53.P$2, J61.P$18, J61.P$19, J98.P$3, R19.2, R22.2, S3.2, U10G$2.VCC, U13G$2.VCC, U8-B.VCC, U9.VDD; no longer C10.2, C11.2, C28.+, J17.P$18, J17.P$19, J44.P$1, J5.P$3, J6-B.P$18, J6-B.P$19, J71.P$1, J73.P$2, J75.P$2, J85.P$2, J92.P$2, R13.2, R3.2, S1.2, U10.VDD, U4-B.VCC, U8G$2.VCC
- net 5V0: now also C6.+, J16.P$3, J20.P$1, J48.P$1, J79.P$5, J79.P$6, J79.P$7, J79.P$8, J92.P$5, J92.P$6, J92.P$7, J92.P$8, J95.P$3, U2.INPUT; no longer C8.+, J4.P$3, J43.P$1, J68.P$1, U3.INPUT
- net 6V0: now also J52.P$1; no longer J42.P$1
- net 9.0V: now also C10.+, J21.P$3, J22.P$3, J23.P$1, U3.INPUT; no longer C6.+, J10.P$3, J2.P$3, J69.P$1, U2.INPUT
- net A2D0: now also J34-A.P$8, J37.P$8, J57.P$1; no longer J16.P$8, J6-A.P$8, J93.P$1
- net A2D1: now also J34-A.P$9, J37.P$9, J56.P$1; no longer J16.P$9, J6-A.P$9, J95.P$1
- net A2D2: now also J34-A.P$10, J37.P$10, J55.P$1; no longer J16.P$10, J6-A.P$10, J94.P$1
- net BATTERY_MOTOR+_IN: now also J44.1@0, J44.1@1, J44.1@2, J44.1@3, J44.1@4, J44.1@5, Q4.D, Q5.D, U11G$1.VDD, U12.COL; no longer J13.1@0, J13.1@1, J13.1@2, J13.1@3, J13.1@4, J13.1@5, Q1.D, Q2.D, U5G$1.VDD, U7.COL
- net BATTERY_MOTOR+_OUT: now also J43.P$1, J44.3@0, J44.3@1, J44.3@2, J44.3@3, J44.3@4, J44.3@5, R13.2, R18.2, U8-A.VIN+; no longer J13.3@0, J13.3@1, J13.3@2, J13.3@3, J13.3@4, J13.3@5, J97.P$1, R11.2, R4.2, U4-A.VIN+
- net BATTERY_MOTOR+_OUT_PRE: now also J42.P$1, Q4.S, Q5.S, R13.1, R16.2, U8-A.VIN-; no longer J96.P$1, Q1.S, Q2.S, R11.1, R5.2, U4-A.VIN-
- net DIO0: now also J34-B.P$1, J61.P$1; no longer J17.P$1, J6-B.P$1
- net DIO1: now also J34-B.P$2, J61.P$2; no longer J17.P$2, J6-B.P$2
- net DIO10: now also J34-B.P$11, J61.P$11; no longer J17.P$11, J6-B.P$11
- net DIO11: now also J34-B.P$12, J61.P$12; no longer J17.P$12, J6-B.P$12
- net DIO2: now also J34-B.P$3, J61.P$3; no longer J17.P$3, J6-B.P$3
- net DIO3: now also J34-B.P$4, J61.P$4; no longer J17.P$4, J6-B.P$4
- net DIO4: now also J34-B.P$5, J61.P$5; no longer J17.P$5, J6-B.P$5
- net DIO5: now also J34-B.P$6, J61.P$6; no longer J17.P$6, J6-B.P$6
- net DIO6: now also J34-B.P$7, J61.P$7; no longer J17.P$7, J6-B.P$7
- net DIO7: now also J34-B.P$8, J61.P$8; no longer J17.P$8, J6-B.P$8
- net DIO8: now also J34-B.P$9, J61.P$9; no longer J17.P$9, J6-B.P$9
- net DIO9: now also J34-B.P$10, J61.P$10; no longer J17.P$10, J6-B.P$10
- net ESC_EN: now also J86.P$2; no longer J29.P$2
- net GND: now also C1.2, C10.-, C11.-, C12.-, C13.-, C14.-, C16.2, C17.2, C18.2, C19.2, C20.2, C23.1, C24.-, C25.2, C26.1, C4.-, J1.P$3, J100.P$3, J2.P$3, J24.P$3, J28.P$2, J3.P$3, J34-B.P$20, J40.P$1, J41.P$2, J44.1@35, J44.1@36, J44.1@37, J44.1@38, J44.1@39, J44.6@0, J44.6@1, J44.6@2, J44.6@3, J44.6@4, J44.6@5, J44.8@5, J51.P$3, J61.P$20, J79.P$1, J79.P$2, J79.P$3, J79.P$4, J9.P$3, J91.P$3, J92.P$1, J92.P$2, J92.P$3, J92.P$4, J99.P$3, R11.1, R12.2, R15.1, R2.2, R3.2, R6.1, S2.P, S3.3, U10G$1.AD0, U10G$1.AD1, U10G$1.AD2, U10G$2.GND, U12.CATH, U13G$2.GND, U5.GND, U5.RES@1, U5.RES@2, U5.RES@3, U5.RES@4, U5.RES@5, U5.RES@6, U6.COM@3, U6.COM@5, U6.COM@6, U6.COM@7, U7.GND, U8-B.GND, U9.AD0, U9.AD1, U9.COM; no longer C1.-, C10.1, C11.1, C16.-, C18.-, C20.-, C23.2, C24.2, C26.-, C27.2, C28.-, C29.2, C30.2, C4.2, C5.-, J11.P$3, J12.P$1, J12.P$2, J12.P$4, J13.1@35, J13.1@36, J13.1@37, J13.1@38, J13.1@39, J13.6@0, J13.6@1, J13.6@2, J13.6@3, J13.6@4, J13.6@5, J13.8@5, J17.P$20, J25.P$3, J45.P$1, J46.P$1, J46.P$2, J46.P$3, J46.P$4, J6-B.P$20, J74.P$2, J8.P$3, J86.P$2, R10.1, R17.2, R19.2, R2.1, R22.2, R7.1, S2.3, S3.P, U10.AD0, U10.AD1, U10.COM, U10.GND, U11.GND, U12.COM@3, U12.COM@5, U12.COM@6, U12.COM@7, U4-B.GND, U7.CATH, U8G$2.GND, U9.RES@1, U9.RES@2, U9.RES@3, U9.RES@4, U9.RES@5, U9.RES@6
- net GND3: now also D1.C, D2.A, J44.2@0, J44.2@1, J44.2@2, J44.2@3, J44.2@4, J44.2@5, J44.4@0, J44.4@1, J44.4@2, J44.4@3, J44.4@4, J44.4@5, J63.P$3, R17.1, R20.1, U11G$1.GND; no longer D1.A, D2.C, J13.2@0, J13.2@1, J13.2@2, J13.2@3, J13.2@4, J13.2@5, J13.4@0, J13.4@1, J13.4@2, J13.4@3, J13.4@4, J13.4@5, J9.P$3, R12.1, R15.1, U5G$1.GND
- net IMOTOR_A2D: now also J54.P$3, J59.P$3, R15.2, U8-A.OUT; no longer J53.P$3, J7.P$3, R10.2, U4-A.OUT
- net N$1: now also R10.1, R11.2, U4.ADJ/GND; no longer R1.1, R2.2, U1.ADJ/GND
- net N$100: now also C16.1, J38.P$1, U6.VS@14, U6.VS@15; no longer C4.1, J92.P$1, U12.VS@14, U12.VS@15
- net N$103: now also C19.1, J55.P$2, U6.ZOUT; no longer C21.1, J93.P$2, U12.ZOUT
- net N$106: now also J20.P$2, R8.2, U3.OUTPUT, U3.VOUT; no longer J68.P$2, R6.2, U2.OUTPUT, U2.VOUT
- net N$107: now also C11.+, J23.P$2, R10.2, U4.OUTPUT, U4.VOUT; no longer C2.+, J69.P$2, R1.2, U1.OUTPUT, U1.VOUT
- net N$109: now also C4.+, J15.P$2, R7.2, U2.OUTPUT, U2.VOUT; no longer C9.+, J71.P$2, R8.2, U3.OUTPUT, U3.VOUT
- net N$110: now also C20.1, J56.P$2, U6.YOUT; no longer C29.1, J95.P$2, U12.YOUT
- net N$111: now also C21.1, J57.P$2, U6.XOUT; no longer C30.1, J94.P$2, U12.XOUT
- net N$12: now also J34-B.P$13, J61.P$13; no longer J17.P$13, J6-B.P$13
- net N$13: now also D4.C, R23.2; no longer J37.P$1
- net N$14: now also J65.P$1; no longer J38.P$1
- net N$15: now also J64.P$1; no longer J39.P$1
- net N$16: now also J34-A.P$2, J37.P$2; no longer J16.P$2, J6-A.P$2
- net N$17: now also J34-A.P$3, J37.P$3; no longer J16.P$3, J6-A.P$3
- net N$18: now also J34-A.P$4, J37.P$4; no longer J16.P$4, J6-A.P$4
- net N$19: now also J34-A.P$5, J37.P$5; no longer J16.P$5, J6-A.P$5
- net N$2: now also S1.1, U1.EN; no longer S2.1, U6.EN
- net N$20: now also J34-A.P$6, J37.P$6; no longer J16.P$6, J6-A.P$6
- net N$21: now also J34-A.P$7, J37.P$7; no longer J16.P$7, J6-A.P$7
- net N$22: now also J34-A.P$11, J37.P$11; no longer J16.P$11, J6-A.P$11
- net N$23: now also J34-A.P$12, J37.P$12; no longer J16.P$12, J6-A.P$12
- net N$24: now also J41.P$1, U7.MODE; no longer J86.P$1, U11.MODE
- net N$25: now also J71.P$1, U9.CH0; no longer J58.P$1, U10.CH0
- net N$26: now also J34-A.P$15, J37.P$15; no longer J16.P$15, J6-A.P$15
- net N$27: now also J34-A.P$16, J37.P$16; no longer J16.P$16, J6-A.P$16
- net N$28: now also C18.1, C22.+, J50.P$1, U5.VDD, U5.VDD_IO; no longer C26.+, C27.1, J73.P$1, U9.VDD, U9.VDD_IO
- net N$29: now also R14.1, U5.CS; no longer R21.1, U9.CS
- net N$3: now also Q4.G, Q5.G, U11G$1.OUT; no longer Q1.G, Q2.G, U5G$1.OUT
- net N$30: now also J34-A.P$19, J37.P$19; no longer J16.P$19, J6-A.P$19
- net N$31: now also J34-A.P$20, J37.P$20; no longer J16.P$20, J6-A.P$20
- net N$32: now also J29.P$1, J30.BACKUPPWR, J30.PWR; no longer J72.BACKUPPWR, J72.PWR, J75.P$1
- net N$33: now also J28.P$1, J30.GND; no longer J72.GND, J74.P$1
- net N$34: now also J27.P$1, J30.STX; no longer J72.STX, J76.P$1
- net N$35: now also J26.P$1, J30.SRX; no longer J72.SRX, J77.P$1
- net N$36: now also J25.P$1, J30.RFBIAS; no longer J72.RFBIAS, J78.P$1
- net N$37: now also C15.2, C17.1, U5.PLLFILT; no longer C24.1, C25.2, U9.PLLFILT
- net N$38: now also C15.1, R12.1; no longer C25.1, R22.1
- net N$39: now also J39.P$3, U5.INT; no longer J80.P$3, U9.INT
- net N$4: now also D1.A, D2.C, R18.1; no longer D1.C, D2.A, R4.1
- net N$40: now also J45.P$3, U5.DRDY/INT2; no longer J79.P$3, U9.DRDY/INT2
- net N$41: now also U9.REF; no longer U10.REF
- net N$42: now also C12.+, C14.+, J10.P$3, J31.P$2, J32.P$2, J33.P$2, R4.1; no longer C20.+, C5.+, J15.P$2, J22.P$3, J81.P$2, J82.P$2, R18.1
- net N$43: now also J53.P$1, U7.3.3V; no longer J85.P$1, U11.3.3V
- net N$44: now also J34-B.P$17, J61.P$17; no longer J17.P$17, J6-B.P$17
- net N$45: now also C2.+, C3.+, U1.VCC; no longer C18.+, C22.+, U6.VCC
- net N$46: now also J36.1, J96.P$1; no longer J14.1, J26.P$1
- net N$47: now also Q1.SA, Q1.SB, Q1.SC, U1.EP, U1.PGND, U1.SGND@1, U1.SGND@2; no longer Q5.SA, Q5.SB, Q5.SC, U6.EP, U6.PGND, U6.SGND@1, U6.SGND@2
- net N$48: now also Q1.G, U1.LG; no longer Q5.G, U6.LG
- net N$49: now also Q2.G, U1.HG; no longer Q4.G, U6.HG
- net N$5: now also R22.1, U12.A, U13G$1.O; no longer R3.1, U7.A, U8G$1.O
- net N$50: now also R3.1; no longer R17.1
- net N$51: now also J4.P$3, R1.2, U1.RON; no longer J20.P$3, R16.2, U6.RON
- net N$52: now also C5.1, J11.P$3, J13.P$3, Q1.DA, Q1.DB, Q1.DC, Q1.DD, Q2.SA, Q2.SB, Q2.SC, R5.2, U1.SW; no longer C19.1, J19.P$3, J54.P$3, Q4.SA, Q4.SB, Q4.SC, Q5.DA, Q5.DB, Q5.DC, Q5.DD, R20.2, U6.SW
- net N$53: now also C5.2, U1.BST; no longer C19.2, U6.BST
- net N$54: now also J6.P$3, J7.P$3, R2.1, R4.2, U1.FB; no longer J23.P$3, J24.P$3, R18.2, R19.1, U6.FB
- net N$55: now also J8.P$3, R5.1, U1.ILIM; no longer J18.P$3, R20.1, U6.ILIM
- net N$56: now also J36.2, J93.P$1; no longer J14.2, J27.P$1
- net N$57: now also J36.3, J89.P$1; no longer J14.3, J28.P$1
- net N$58: now also C1.1, U1.SS; no longer C23.1, U6.SS
- net N$59: now also J36.4, J86.P$1; no longer J14.4, J29.P$1
- net N$60: now also J36.5, J83.P$1; no longer J14.5, J30.P$1
- net N$61: now also J36.6, J80.P$1; no longer J14.6, J31.P$1
- net N$62: now also J36.7, J76.P$1; no longer J14.7, J32.P$1
- net N$63: now also J36.8, J73.P$1; no longer J14.8, J33.P$1
- net N$64: now also J36.9, J70.P$1; no longer J14.9, J34.P$1
- net N$65: now also J36.10, J68.P$1; no longer J14.10, J35.P$1
- net N$66: now also J60.P$1; no longer J40.P$1
- net N$67: now also J58.P$1; no longer J41.P$1
- net N$68: now also J36.20, J67.P$2; no longer J14.20, J36.P$2
- net N$69: now also J36.19, J66.P$2; no longer J14.19, J37.P$2
- net N$70: now also J36.18, J65.P$2; no longer J14.18, J38.P$2
- net N$71: now also J36.17, J64.P$2; no longer J14.17, J39.P$2
- net N$72: now also J36.16, J60.P$2; no longer J14.16, J40.P$2
- net N$73: now also J36.15, J58.P$2; no longer J14.15, J41.P$2
- net N$74: now also J36.14, J52.P$2; no longer J14.14, J42.P$2
- net N$75: now also J36.13, J48.P$2; no longer J14.13, J43.P$2
- net N$76: now also J36.12, J46.P$2; no longer J14.12, J44.P$2
- net N$77: now also J36.11, J40.P$2; no longer J14.11, J45.P$2
- net N$78: now also J97.P$1, R21.1, U13G$1.I1; no longer J47.P$1, R13.1, U8G$1.I1
- net N$79: now also R20.2, U11G$1.IN, U12.E; no longer R12.2, U5G$1.IN, U7.E
- net N$8: now also S3.1, U13G$1.I0; no longer S1.1, U8G$1.I0
- net N$80: now also J34-B.P$16, J61.P$16; no longer J17.P$16, J6-B.P$16
- net N$85: now also J49.P$1, U7.TX; no longer J84.P$1, U11.TX
- net N$86: now also J47.P$1, U7.RX; no longer J83.P$1, U11.RX
- net N$87: now also J74.P$1, U9.CH1; no longer J59.P$1, U10.CH1
- net N$9: now also R19.1; no longer R14.1
- net N$90: now also J77.P$1, U9.CH2; no longer J60.P$1, U10.CH2
- net N$91: now also J81.P$1, U9.CH3; no longer J87.P$1, U10.CH3
- net N$96: now also J84.P$1, U9.CH4; no longer J88.P$1, U10.CH4
- net N$97: now also J87.P$1, U9.CH5; no longer J89.P$1, U10.CH5
- net N$98: now also U9.CH6; no longer U10.CH6
- net N$99: now also J94.P$1, U9.CH7; no longer J91.P$1, U10.CH7
- net POWER_LIPO+_IN: now also J44.7@0, J44.7@1, J44.7@2, J44.7@3, J44.7@4, J44.7@5; no longer J13.7@0, J13.7@1, J13.7@2, J13.7@3, J13.7@4, J13.7@5
- net POWER_LIPO_POST: now also C8.+, C9.+, J5.P$3, Q2.DA, Q2.DB, Q2.DC, Q2.DD, R1.1, U1.VIN; no longer C16.+, C3.+, J21.P$3, Q4.DA, Q4.DB, Q4.DC, Q4.DD, R16.1, U6.VIN
- net QUAD0A: now also J83.P$2; no longer J30.P$2
- net QUAD0B: now also J80.P$2; no longer J31.P$2
- net QUAD1A: now also J76.P$2; no longer J32.P$2
- net QUAD1B: now also J73.P$2; no longer J33.P$2
- net SCL: now also J34-B.P$15, J61.P$15, J68.P$2, J85.P$3, U10G$1.SCL, U5.SCL/SPC, U9.SCL; no longer J17.P$15, J35.P$2, J6-B.P$15, U10.SCL, U9.SCL/SPC
- net SDA: now also J34-B.P$14, J61.P$14, J70.P$2, J88.P$3, U10G$1.SDA, U5.SDA/SDI/SDO, U9.SDA; no longer J17.P$14, J34.P$2, J6-B.P$14, U10.SDA, U9.SDA/SDI/SDO
- net SPM2: now also J89.P$2; no longer J28.P$2
- net SPWM0: now also J96.P$2; no longer J26.P$2
- net SPWM1: now also J93.P$2; no longer J27.P$2
- net SRX0: now also J27.P$2, J34-A.P$17, J37.P$17; no longer J16.P$17, J6-A.P$17, J76.P$2
- net SRX1: now also J34-A.P$13, J37.P$13, J49.P$2; no longer J16.P$13, J6-A.P$13, J84.P$2
- net STX0: now also J26.P$2, J34-A.P$18, J37.P$18; no longer J16.P$18, J6-A.P$18, J77.P$2
- net STX1: now also J34-A.P$14, J37.P$14, J47.P$2; no longer J16.P$14, J6-A.P$14, J83.P$2
- net VMOTOR_A2D: now also J62.P$3, R16.1, R17.2; no longer J3.P$3, R15.2, R5.1

Commit message: updated part numbers
Parts:
- R10: value ERJ-3EKF1780V -> PRESI00039; device aAcroname:ERJ-3EKF1780V -> aAcroname:PRESI00039; ACRONAME (none) -> PRESI00039; PARTNUM (none) -> ERJ-3EKF6980V
- R11: device aAcroname:ERJ-3EKF3830V -> aAcroname:RESISTOR; RESISTANCE (none) -> 4.22k
- R6: device aAcroname:ERJ-3EKF3830V -> aAcroname:PRESI00002; ACRONAME (none) -> PRESI00002; PARTNUM (none) -> ERJ-3GEYJ332V
- R7: value ERJ-3EKF1780V -> PRESI00007; device aAcroname:ERJ-3EKF1780V -> aAcroname:PRESI00007; ACRONAME (none) -> PRESI00007; PARTNUM (none) -> ERJ-3GEYJ222V
- R8: value ERJ-3EKF1780V -> PRESI00019; device aAcroname:ERJ-3EKF1780V -> aAcroname:PRESI00019; ACRONAME (none) -> PRESI00019; PARTNUM (none) -> ERJ-3EKF2431V
- R9: device aAcroname:ERJ-3EKF3830V -> aAcroname:PRESI00056; ACRONAME (none) -> PRESI00056; PARTNUM (none) -> ERJ-3EKF6491V
Other:
- note added: "12.0 V LDO calculations Calculating resitor values for LDO for 12.000V. Tried 4683 resistor combinations. Final Voltage of: 11.996 using R1: 330.0 ohm R2: 2800.0 ohm Acroname Stock Part. Use R1 = PRESI00060 (330.000 ohm) Voutput range w/ 1 percent: 11.785V - 12.212V 9.0 V LDO calculations Calculating resitor values for LDO for 9.000V. Tried 4683 resistor combinations. Final Voltage of: 9.018 usin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"
- moved on the sheet: R6, R9
Changed lines of the file:
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@@
 <attribute name="ACRONAME" value="PCAPI00037"/>
 </part>
-<part name="R10" library="aAcroname" deviceset="ERJ-3EKF1780V" device=""/>
-<part name="R11" library="aAcroname" deviceset="ERJ-3EKF3830V" device="" value="on"/>
+<part name="R10" library="aAcroname" deviceset="PRESI00039" device="">
+<attribute name="ACRONAME" value="PRESI00039"/>
+<attribute name="PARTNUM" value="ERJ-3EKF6980V"/>
+</part>
+<part name="R11" library="aAcroname" deviceset="RESISTOR" device="" value="on">
+<attribute name="PARTNUM" value=""/>
+<attribute name="RESISTANCE" value="4.22k"/>
+</part>
 <part name="C11" library="aAcroname" deviceset="T491D227K016ZT" device="">
 <attribute name="ACRONAME" value="PCAPI00037"/>
@@
 <attribute name="ACRONAME" value="PCAPI00037"/>
 </part>
-<part name="R8" library="aAcroname" deviceset="ERJ-3EKF1780V" device=""/>
-<part name="R9" library="aAcroname" deviceset="ERJ-3EKF3830V" device="" value="on"/>
+<part name="R8" library="aAcroname" deviceset="PRESI00019" device="">
+<attribute name="ACRONAME" value="PRESI00019"/>
+<attribute name="PARTNUM" value="ERJ-3EKF2431V"/>
+</part>
+<part name="R9" library="aAcroname" deviceset="PRESI00056" device="" value="on">
+<attribute name="ACRONAME" value="PRESI00056"/>
+<attribute name="PARTNUM" value="ERJ-3EKF6491V"/>
+</part>
 <part name="C7" library="aAcroname" deviceset="T491D227K016ZT" device="">
 <attribute name="ACRONAME" value="PCAPI00037"/>
@@
 <attribute name="ACRONAME" value="PCAPI00037"/>
 </part>
-<part name="R7" library="aAcroname" deviceset="ERJ-3EKF1780V" device=""/>
-<part name="R6" library="aAcroname" deviceset="ERJ-3EKF3830V" device="" value="on"/>
+<part name="R7" library="aAcroname" deviceset="PRESI00007" device="">
+<attribute name="ACRONAME" value="PRESI00007"/>
+<attribute name="PARTNUM" value="ERJ-3GEYJ222V"/>
+</part>
+<part name="R6" library="aAcroname" deviceset="PRESI00002" device="" value="on">
+<attribute name="ACRONAME" value="PRESI00002"/>
+<attribute name="PARTNUM" value="ERJ-3GEYJ332V"/>
+</part>
 <part name="C4" library="aAcroname" deviceset="T491D227K016ZT" device="">
 <attribute name="ACRONAME" value="PCAPI00037"/>
@@
 <text x="170.18" y="172.72" size="1.778" layer="97">Don't forget to adjust feedback resistor values!!!</text>
 <rectangle x1="183.388" y1="10.16" x2="219.964" y2="16.51" layer="105"/>
+<text x="7.62" y="157.48" size="1.778" layer="97">12.0 V LDO calculations Calculating resitor values for LDO for 12.000V. Tried 4683 resistor combinations. Final Voltage of: 11.996 using R1: 330.0 ohm  R2: 2800.0 ohm   Acroname Stock Part. Use R1 = PRESI00060 (330.000 ohm)   Voutput range w/ 1 percent: 11.785V - 12.212V  9.0 V LDO calculations Calculating resitor values for LDO for 9.000V. Tried 4683 resistor combinations. Final Voltage of: 9.018 using R1: 698.0 ohm  R2: 4220.0 ohm   Acroname Stock Part. Use R1 = PRESI00039 (698.000 ohm)   Voutput range w/ 1 percent: 8.867V - 9.173V  5.0 V LDO calculations Calculating resitor values for LDO for 5.000V. Tried 441 resistor combinations. Final Voltage of: 4.955 using R1: 2400.0 ohm  R2: 6490.0 ohm   Acroname Stock Part. Use R1 = PRESI00019 (2400.000 ohm)   Acroname Stock Part. Use R2 = PRESI00056 (6490.000 ohm)   Voutput range w/ 1 percent: 4.885V - 5.026V  3.3 V LDO calculations Calculating resitor values for LDO for 3.300V. Tried 441 resistor combinations. Final Voltage of: 3.290 using R1: 2200.0 ohm  R2: 3300.0 ohm   Acroname Stock Part. Use R1 = PRESI00007 (2200.000 ohm)   Acroname Stock Part. \nUse R2 = PRESI00002 (3300.000 ohm)   Voutput range w/ 1 percent: 3.251V - 3.330V</text>
 </plain>
 <instances>
@@
 <attribute name="NAME" x="97.5614" y="79.756" size="1.27" layer="95" rot="R90"/>
 <attribute name="NOTES" x="103.9114" y="78.486" size="1.27" layer="95" rot="R90"/>
+<attribute name="RESISTANCE" x="101.854" y="77.724" size="1.27" layer="96" font="vector" rot="R90"/>
 </instance>
 <instance part="C11" gate="G$1" x="106.68" y="101.6"/>

Commit message: checking in schematic changes
Parts:
- J100, J12, J14, J17, J19, J2, J3, J9, J98, J99: NOTES No Stuff -> (none)
- J34: ALTERNATIVE (none) -> SSW-120-01-G-S:75915-320LF; PARTNUM (none) -> 1-534237-8
Other:
- note added: "12.0 V LDO: Final Voltage of: 11.996 using R1: 330.0 ohm R2: 2800.0 ohm Acroname Stock Part. Use R1 = PRESI00060 (330.000 ohm)"
- note added: "3.3 V LDO: Final Voltage of: 3.290 using R1: 2200.0 ohm R2: 3300.0 ohm Acroname Stock Part. Use R1 = PRESI00007 (2200.000 ohm) Acroname Stock Part. Use R2 = PRESI00002 (3300.000 ohm)"
- note added: "5.0 V LDO: Final Voltage of: 4.955 using R1: 2400.0 ohm R2: 6490.0 ohm Acroname Stock Part. Use R1 = PRESI00019 (2400.000 ohm) Acroname Stock Part. Use R2 = PRESI00056 (6490.000 ohm)"
- note added: "9.0 V LDO: Final Voltage of: 9.018 using R1: 698.0 ohm R2: 4220.0 ohm Acroname Stock Part. Use R1 = PRESI00039 (698.000 ohm)"
- note removed: "12.0 V LDO calculations Calculating resitor values for LDO for 12.000V. Tried 4683 resistor combinations. Final Voltage of: 11.996 using R1: 330.0 ohm R2: 2800.0 ohm Acroname Stock Part. Use R1 = PRESI00060 (330.000 ohm) Voutput range w/ 1 percent: 11.785V - 12.212V 9.0 V LDO calculations Calculating resitor values for LDO for 9.000V. Tried 4683 resistor combinations. Final Voltage of: 9.018 usin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"
- note removed: "Don't forget to adjust feedback resistor values!!!"
